Commit message: Improve contact computation during retargeting and add successful RL MDP

File: robotic_grounding/source/robotic_grounding/robotic_grounding/assets/urdfs/arctic/box.urdf (robot description, URDF)
Before this commit: robot box, 8 links, 7 joints
Links:
- removed link base
- removed link base_pitch
- removed link base_roll
- removed link base_x
- removed link base_y
- removed link base_z
Joints:
- removed joint base_pitch
- removed joint base_roll
- removed joint base_x
- removed joint base_y
- removed joint base_yaw
- removed joint base_z
