Commit message: Change table assets and add simple box mesh

File: robotic_grounding/source/robotic_grounding/robotic_grounding/assets/urdfs/arctic/box_rigid.urdf (robot description, URDF)
Before this commit: robot box, 1 links, 0 joints
Links:
- link object: geometry collision mesh filename=../../meshes/arctic/box/mesh_tex_simple.obj scale=0.001 0.001 0.001; visual mesh filename=../../meshes/arctic/box/mesh_tex.obj scale=0.001 0.001 0.001

Commit message: Add task composer, modify command class, and relative hand keypoints for multiple rigid and articulated objects

File: robotic_grounding/source/robotic_grounding/robotic_grounding/assets/urdfs/arctic/box_rigid.urdf (robot description, URDF)
Before this commit: robot box, 1 links, 0 joints
Links:
- link object: geometry collision mesh filename=../../meshes/arctic/box/mesh_tex_tiny.obj scale=1 1 1; visual mesh filename=../../meshes/arctic/box/mesh_tex_tiny.obj scale=1 1 1
