Commit message: add contact wrench space support rewards

File: robotic_grounding/source/robotic_grounding/robotic_grounding/assets/urdfs/arctic/capsulemachine_rigid.urdf (robot description, URDF)
Before this commit: robot capsulemachine, 1 links, 0 joints
Links:
- link object: mass 1.048362679505015 -> 0.3

File: robotic_grounding/source/robotic_grounding/robotic_grounding/assets/urdfs/arctic/espressomachine_rigid.urdf (robot description, URDF)
Before this commit: robot espressomachine, 1 links, 0 joints
Links:
- link object: mass 1.892773469188377 -> 0.3

File: robotic_grounding/source/robotic_grounding/robotic_grounding/assets/urdfs/arctic/ketchup_rigid.urdf (robot description, URDF)
Before this commit: robot ketchup, 1 links, 0 joints
Links:
- link object: mass 0.5700573317889485 -> 0.3

File: robotic_grounding/source/robotic_grounding/robotic_grounding/assets/urdfs/arctic/laptop_rigid.urdf (robot description, URDF)
Before this commit: robot laptop, 1 links, 0 joints
Links:
- link object: mass 0.9048766224119441 -> 0.3

File: robotic_grounding/source/robotic_grounding/robotic_grounding/assets/urdfs/arctic/mixer_rigid.urdf (robot description, URDF)
Before this commit: robot mixer, 1 links, 0 joints
Links:
- link object: mass 0.5896949643710692 -> 0.3

File: robotic_grounding/source/robotic_grounding/robotic_grounding/assets/urdfs/arctic/notebook_rigid.urdf (robot description, URDF)
Before this commit: robot notebook, 1 links, 0 joints
Links:
- link object: mass 0.7669728222307014 -> 0.3

File: robotic_grounding/source/robotic_grounding/robotic_grounding/assets/urdfs/sharpawave/left_sharpa_wave.urdf (robot description, URDF)
Before this commit: robot dual_sharpa_wave, 33 links, 32 joints
Links:
- link left_hand_C_MC: geometry collision mesh filename=../meshes/sharpa_wave/left_cvx/left_hand_C_MC_cut.STL; visual mesh filename=../meshes/sharpa_wave/left_cvx/left_hand_C_MC_visual_.STL
- link left_thumb_MC: geometry collision mesh filename=../meshes/sharpa_wave/left_cvx/left_thumb_MC_cut.STL; visual mesh filename=../meshes/sharpa_wave/left_cvx/left_thumb_MC_visual.STL

File: robotic_grounding/source/robotic_grounding/robotic_grounding/assets/urdfs/sharpawave/right_sharpa_wave.urdf (robot description, URDF)
Before this commit: robot right_sharpa_wave, 33 links, 32 joints
Links:
- link right_hand_C_MC: geometry collision mesh filename=../meshes/sharpa_wave/right_cvx/right_hand_C_MC_cut.STL; visual mesh filename=../meshes/sharpa_wave/right_cvx/right_hand_C_MC_visual_.STL
- link right_thumb_MC: geometry collision mesh filename=../meshes/sharpa_wave/right_cvx/right_thumb_MC_cut.STL; visual mesh filename=../meshes/sharpa_wave/right_cvx/right_thumb_MC_visual.STL
