Commit message: fix articulated voc and torque compensation

File: robotic_grounding/source/robotic_grounding/robotic_grounding/assets/urdfs/arctic/capsulemachine_art.urdf (robot description, URDF)
Before this commit: robot capsulemachine, 2 links, 1 joints
Joints:
- joint rotation: limit lower=0 upper=3.141592653589793 effort=1000 velocity=200 -> lower=0 upper=1.92 effort=1000 velocity=200
