Commit message: update arctic urdf joint limits

File: robotic_grounding/source/robotic_grounding/robotic_grounding/assets/urdfs/arctic/box_art.urdf (robot description, URDF)
Before this commit: robot box, 2 links, 1 joints
Joints:
- joint rotation: limit lower=0 upper=3.141592653589793 effort=1000 velocity=200 -> lower=0 upper=2.305 effort=1000 velocity=200

File: robotic_grounding/source/robotic_grounding/robotic_grounding/assets/urdfs/arctic/capsulemachine_art.urdf (robot description, URDF)
Before this commit: robot capsulemachine, 2 links, 1 joints
Joints:
- joint rotation: limit lower=0 upper=1.92 effort=1000 velocity=200 -> lower=0 upper=1.82 effort=1000 velocity=200

File: robotic_grounding/source/robotic_grounding/robotic_grounding/assets/urdfs/arctic/espressomachine_art.urdf (robot description, URDF)
Before this commit: robot espressomachine, 2 links, 1 joints
Joints:
- joint rotation: limit lower=0 upper=1.5 effort=1000 velocity=200 -> lower=0 upper=1.525 effort=1000 velocity=200

File: robotic_grounding/source/robotic_grounding/robotic_grounding/assets/urdfs/arctic/ketchup_art.urdf (robot description, URDF)
Before this commit: robot ketchup, 2 links, 1 joints
Joints:
- joint rotation: limit lower=0 upper=2.5 effort=1000 velocity=200 -> lower=0 upper=3.785 effort=1000 velocity=200

File: robotic_grounding/source/robotic_grounding/robotic_grounding/assets/urdfs/arctic/laptop_art.urdf (robot description, URDF)
Before this commit: robot laptop, 2 links, 1 joints
Joints:
- joint rotation: limit lower=0 upper=3.141592653589793 effort=1000 velocity=200 -> lower=0 upper=2.354 effort=1000 velocity=200

File: robotic_grounding/source/robotic_grounding/robotic_grounding/assets/urdfs/arctic/microwave_art.urdf (robot description, URDF)
Before this commit: robot microwave, 2 links, 1 joints
Joints:
- joint rotation: limit lower=0 upper=3.141592653589793 effort=1000 velocity=200 -> lower=0 upper=1.736 effort=1000 velocity=200

File: robotic_grounding/source/robotic_grounding/robotic_grounding/assets/urdfs/arctic/mixer_art.urdf (robot description, URDF)
Before this commit: robot mixer, 2 links, 1 joints
Joints:
- joint rotation: limit lower=0 upper=3.141592653589793 effort=1000 velocity=200 -> lower=0 upper=1.688 effort=1000 velocity=200

File: robotic_grounding/source/robotic_grounding/robotic_grounding/assets/urdfs/arctic/notebook_art.urdf (robot description, URDF)
Before this commit: robot notebook, 2 links, 1 joints
Joints:
- joint rotation: limit lower=0 upper=3.141592653589793 effort=1000 velocity=200 -> lower=0 upper=3.144 effort=1000 velocity=200

File: robotic_grounding/source/robotic_grounding/robotic_grounding/assets/urdfs/arctic/phone_art.urdf (robot description, URDF)
Before this commit: robot phone, 2 links, 1 joints
Joints:
- joint rotation: limit lower=0 upper=2.5 effort=1000 velocity=200 -> lower=0 upper=3.027 effort=1000 velocity=200

File: robotic_grounding/source/robotic_grounding/robotic_grounding/assets/urdfs/arctic/waffleiron_art.urdf (robot description, URDF)
Before this commit: robot waffleiron, 2 links, 1 joints
Joints:
- joint rotation: limit lower=0 upper=3.141592653589793 effort=1000 velocity=200 -> lower=0 upper=2.954 effort=1000 velocity=200
