Commit message: fix primitive sharpa urdfs

File: robotic_grounding/source/robotic_grounding/robotic_grounding/assets/urdfs/sharpawave/left_sharpa_wave_primitive.urdf (robot description, URDF)
Before this commit: robot dual_sharpa_wave, 33 links, 32 joints
Links:
- link left_hand_C_MC: geometry collision capsule length=0.013 radius=0.0209; collision capsule length=0.035 radius=0.0209
- link left_index_MCP_VL: geometry collision sphere radius=0.009; visual mesh filename=../meshes/sharpa_wave/left_cvx/left_MCP_VL_visual.STL
- link left_middle_MCP_VL: geometry collision sphere radius=0.009; visual mesh filename=../meshes/sharpa_wave/left_cvx/left_MCP_VL_visual.STL
- link left_pinky_MC: geometry collision capsule length=0.02446 radius=0.01228; collision capsule length=0.02446 radius=0.01228
- link left_pinky_MCP_VL: geometry collision sphere radius=0.009; visual mesh filename=../meshes/sharpa_wave/left_cvx/left_MCP_VL_visual.STL
- link left_ring_MCP_VL: geometry collision sphere radius=0.009; visual mesh filename=../meshes/sharpa_wave/left_cvx/left_MCP_VL_visual.STL

File: robotic_grounding/source/robotic_grounding/robotic_grounding/assets/urdfs/sharpawave/right_sharpa_wave_primitive.urdf (robot description, URDF)
Before this commit: robot right_sharpa_wave, 33 links, 32 joints
Links:
- link right_hand_C_MC: geometry collision capsule length=0.013 radius=0.0209; collision capsule length=0.035 radius=0.0209
- link right_index_MCP_VL: geometry collision sphere radius=0.009; visual mesh filename=../meshes/sharpa_wave/right_cvx/right_MCP_VL_visual.STL
- link right_middle_MCP_VL: geometry collision sphere radius=0.009; visual mesh filename=../meshes/sharpa_wave/right_cvx/right_MCP_VL_visual.STL
- link right_pinky_MC: geometry collision capsule length=0.02446 radius=0.01228; collision capsule length=0.02446 radius=0.01228
- link right_pinky_MCP_VL: geometry collision sphere radius=0.009; visual mesh filename=../meshes/sharpa_wave/right_cvx/right_MCP_VL_visual.STL
- link right_ring_MCP_VL: geometry collision sphere radius=0.009; visual mesh filename=../meshes/sharpa_wave/right_cvx/right_MCP_VL_visual.STL
