Commit message: add mano to dex3 retargeting (arctic + taco) + --robot dispatch

File: robotic_grounding/source/robotic_grounding/robotic_grounding/assets/urdfs/g1/dex3_left.urdf (robot description, URDF)
Before this commit: robot dex3_left_hand, 18 links, 17 joints
Links:
- removed link base_pitch_link
- removed link base_roll_link
- removed link base_x_link
- removed link base_y_link
- removed link base_yaw_link
- removed link base_z_link
- removed link world
Joints:
- removed joint base_pitch_joint
- removed joint base_roll_joint
- removed joint base_x_joint
- removed joint base_y_joint
- removed joint base_yaw_joint
- removed joint base_z_joint
- removed joint left_hand_palm_joint

File: robotic_grounding/source/robotic_grounding/robotic_grounding/assets/urdfs/g1/dex3_right.urdf (robot description, URDF)
Before this commit: robot dex3_right_hand, 18 links, 17 joints
Links:
- removed link base_pitch_link
- removed link base_roll_link
- removed link base_x_link
- removed link base_y_link
- removed link base_yaw_link
- removed link base_z_link
- removed link world
Joints:
- removed joint base_pitch_joint
- removed joint base_roll_joint
- removed joint base_x_joint
- removed joint base_y_joint
- removed joint base_yaw_joint
- removed joint base_z_joint
- removed joint right_hand_palm_joint

Commit message: Clean up planner and Sonic assets

File: robotic_grounding/source/robotic_grounding/robotic_grounding/assets/urdfs/g1/dex3_left.urdf (robot description, URDF)
Before this commit: robot dex3_left, 11 links, 10 joints
Links:
- link left_hand_index_0_link: geometry collision mesh filename=package://g1/left_hand_index_0_link.STL; visual mesh filename=package://g1/left_hand_index_0_link.STL
- link left_hand_index_1_link: geometry collision mesh filename=package://g1/left_hand_index_1_link.STL; visual mesh filename=package://g1/left_hand_index_1_link.STL
- link left_hand_middle_0_link: geometry collision mesh filename=package://g1/left_hand_middle_0_link.STL; visual mesh filename=package://g1/left_hand_middle_0_link.STL
- link left_hand_middle_1_link: geometry collision mesh filename=package://g1/left_hand_middle_1_link.STL; visual mesh filename=package://g1/left_hand_middle_1_link.STL
- link left_hand_palm_link: geometry collision mesh filename=package://g1/left_hand_palm_link.STL; visual mesh filename=package://g1/left_hand_palm_link.STL
- link left_hand_thumb_0_link: geometry collision mesh filename=package://g1/collision/hands/left_hand_thumb_0_link.obj; visual mesh filename=package://g1/left_hand_thumb_0_link.STL
- link left_hand_thumb_1_link: geometry collision mesh filename=package://g1/collision/hands/left_hand_thumb_1_link.obj; visual mesh filename=package://g1/left_hand_thumb_1_link.STL
- link left_hand_thumb_2_link: geometry collision mesh filename=package://g1/collision/hands/left_hand_thumb_2_link.obj; visual mesh filename=package://g1/left_hand_thumb_2_link.STL

File: robotic_grounding/source/robotic_grounding/robotic_grounding/assets/urdfs/g1/dex3_right.urdf (robot description, URDF)
Before this commit: robot dex3_right, 11 links, 10 joints
Links:
- link right_hand_index_0_link: geometry collision mesh filename=package://g1/right_hand_index_0_link.STL; visual mesh filename=package://g1/right_hand_index_0_link.STL
- link right_hand_index_1_link: geometry collision mesh filename=package://g1/right_hand_index_1_link.STL; visual mesh filename=package://g1/right_hand_index_1_link.STL
- link right_hand_middle_0_link: geometry collision mesh filename=package://g1/right_hand_middle_0_link.STL; visual mesh filename=package://g1/right_hand_middle_0_link.STL
- link right_hand_middle_1_link: geometry collision mesh filename=package://g1/right_hand_middle_1_link.STL; visual mesh filename=package://g1/right_hand_middle_1_link.STL
- link right_hand_palm_link: geometry collision mesh filename=package://g1/right_hand_palm_link.STL; visual mesh filename=package://g1/right_hand_palm_link.STL
- link right_hand_thumb_0_link: geometry collision mesh filename=package://g1/collision/hands/right_hand_thumb_0_link.obj; visual mesh filename=package://g1/right_hand_thumb_0_link.STL
- link right_hand_thumb_1_link: geometry collision mesh filename=package://g1/collision/hands/right_hand_thumb_1_link.obj; visual mesh filename=package://g1/right_hand_thumb_1_link.STL
- link right_hand_thumb_2_link: geometry collision mesh filename=package://g1/collision/hands/right_hand_thumb_2_link.obj; visual mesh filename=package://g1/right_hand_thumb_2_link.STL
